Commit message: Adapt midterm URDF to match tutorial robot

File: gazebo_controller/launch/building_robot.urdf (robot description, URDF)
Before this commit: robot basic_robot, 4 links, 3 joints
Links:
- removed link lidar_dome
- added link base_link
- added link caster; visual sphere radius=0.2
- link chassis: geometry visual box size=2.0 1.0 0.5
- link left_wheel: geometry visual cylinder length=0.2 radius=0.4
- link right_wheel: geometry visual cylinder length=0.2 radius=0.4
Joints:
- removed joint chassis_to_lidar_dome
- added joint base_link_to_chassis: type fixed, parent base_link, child chassis, origin xyz=0.5 0 0.4 rpy=0 0 0
- added joint chassis_to_caster: type fixed, parent chassis, child caster, origin xyz=0.8 0 -0.2 rpy=0 0 0
- joint chassis_to_left_wheel: axis 0 0 1 -> (none); origin xyz=0 0.4375 0 rpy=1.57075 0 0 -> xyz=-0.5 0.6 0 rpy=1.57075 0 0; type continuous -> fixed
- joint chassis_to_right_wheel: axis 0 0 1 -> (none); origin xyz=0 -0.4375 0 rpy=1.57075 0 0 -> xyz=-0.5 -0.6 0 rpy=1.57075 0 0; type continuous -> fixed
